Commit message: 👌 IMPROVE:  refactoring

File: robot_table_control/urdf/robot_table_controlled.urdf.xacro (robot description, xacro)
@@ -6,6 +6,4 @@
   <xacro:include filename="$(find ur_robot_driver)/urdf/ur.ros2_control.xacro"/>
   <xacro:include filename="$(find robotiq_description)/urdf/2f_85.ros2_control.xacro"/>
-  <!--<xacro:include filename="$(find robotiq_description)/urdf/ur_to_robotiq_adapter.urdf.xacro"/>-->
-  <!--<xacro:include filename="$(find robotiq_description)/urdf/robotiq_2f_85_macro.urdf.xacro"/>-->
   <!--We need to specify the arguments used for parametrizing our description-->
   <xacro:arg name="ur_type" default="ur5e"/>

File: robot_table_description/urdf/robot_table.urdf.xacro (robot description, xacro)
@@ -22,12 +22,3 @@
       <origin xyz="0 0 0.77526" rpy="0 0 0" />
   </xacro:robot_table>
-  <!--<xacro:robotiq_gripper
-    name="RobotiqGripper"
-    prefix=""
-    parent="ur5e_tool0"
-    com_port="/tmp/ttyUR"
-    use_fake_hardware="false"
-    include_ros2_control="true">
-    <origin xyz="0 0 0" rpy="0 0 0" />
-</xacro:robotiq_gripper>-->
 </robot>

Commit message: 👌 IMPROVE: update robot table

File: robot_table_control/urdf/robot_table_controlled.urdf.xacro (robot description, xacro)
@@ -30,5 +30,6 @@
     visual_parameters_file="$(arg visual_parameters_file)"
   >
-    <origin xyz="0 0 0.77526" rpy="0 0 0" />
+    <!--<origin xyz="0 0 0.77526" rpy="0 0 0" />-->
+    <origin xyz="0 0 0.71676" rpy="0 0 0" />
   </xacro:robot_table>
   <!--Create the control tag for the UR robot-->

File: robot_table_description/urdf/robot_table.urdf.xacro (robot description, xacro)
@@ -20,5 +20,6 @@
     visual_parameters_file="$(arg visual_parameters_file)"
     >
-      <origin xyz="0 0 0.77526" rpy="0 0 0" />
+      <!--<origin xyz="0 0 0.77526" rpy="0 0 0" />-->
+      <origin xyz="0 0 0.71676" rpy="0 0 0" />
   </xacro:robot_table>
 </robot>

File: robot_table_description/urdf/robot_table_macro.xacro (robot description, xacro)
@@ -24,5 +24,6 @@
           <mesh filename="package://robot_table_description/meshes/robo_table.dae"/>
         </geometry>
-        <origin xyz="0 0 -0.01" rpy="${pi/2} 0 0"/>
+        <!--<origin xyz="0 0 -0.01" rpy="${pi/2} 0 0"/>-->
+        <origin xyz="0 0 0" rpy="${pi/2} 0 0"/>
       </visual>
       <collision>
@@ -31,5 +32,6 @@
           <mesh filename="package://robot_table_description/meshes/robo_table.dae"/>
         </geometry>
-        <origin xyz="0 0 -0.01" rpy="${pi/2} 0 0"/>
+        <!--<origin xyz="0 0 -0.01" rpy="${pi/2} 0 0"/>-->
+        <origin xyz="0 0 0" rpy="${pi/2} 0 0"/>
       </collision>
     </link>
@@ -38,5 +40,5 @@
       <parent link="table"/>
       <child link="robot_mount"/>
-      <origin xyz="0 0 0" rpy="0 0 0" />
+      <origin xyz="0 0 0.02" rpy="0 0 0" />
     </joint>
     <!--This will create the specific robot-->
@@ -65,4 +67,27 @@
     include_ros2_control="false">
     <origin xyz="0 0 0" rpy="0 0 0"/>
-</xacro:robotiq_gripper>
+  </xacro:robotiq_gripper>
+<!--<link name="camera_link">
+  <visual>
+    <geometry>
+      <mesh filename="package://robot_table_description/meshes/intel_realsense_d415.dae"/>
+    </geometry>
+  </visual>
+  <collision>
+    <geometry>
+      <mesh filename="package://robot_table_description/meshes/intel_realsense_d415.dae"/>
+    </geometry>
+  </collision>
+  <inertial>
+    <mass value="0.01"/>
+    <origin xyz="0 0 0"/>
+    <inertia ixx="1e-6" iyy="1e-6" izz="1e-6"
+             ixy="0" ixz="0" iyz="0"/>
+  </inertial>
+</link>
+<joint name="camera_joint" type="fixed">
+  <parent link="ur5e_tool0"/>
+  <child link="camera_link"/>
+  <origin xyz="0.1 0.1 0.1" rpy="-${pi/2} 0 0"/>
+</joint>-->
 </robot>

File: robot_table_gazebo/urdf/ur_gz.urdf.xacro (robot description, xacro)
@@ -101,3 +101,26 @@
     <origin xyz="0 0 0" rpy="0 0 0" />
   </xacro:robotiq_gripper>
+<!--ros2 camera instance -->
+<!--<gazebo reference="camera_link">
+  <sensor name="camera_link" type="depth_camera">
+    <always_on>1</always_on>
+    <update_rate>30</update_rate>
+    <visualize>true</visualize>
+    <topic>depth_camera</topic>
+    <camera>
+      <horizontal_fov>1.211</horizontal_fov>
+      <image>
+        <width>640</width>
+        <height>480</height>
+      </image>
+      <clip>
+        <near>0.05</near>
+        <far>10.0</far>
+      </clip>
+    </camera>
+    <plugin name="gz::sim::systems::Sensors"
+            filename="gz-sim-sensors-system">
+    </plugin>
+  </sensor>
+</gazebo> -->
 </robot>
