Commit message: 👌 IMPROVE: refactoring

File: robot_table_description/urdf/robot_table.urdf.xacro (robot description, xacro)
@@ -20,5 +20,4 @@
     visual_parameters_file="$(arg visual_parameters_file)"
     >
-      <!--<origin xyz="0 0 0.77526" rpy="0 0 0" />-->
       <origin xyz="0 0 0.71676" rpy="0 0 0" />
   </xacro:robot_table>

File: robot_table_description/urdf/robot_table_macro.xacro (robot description, xacro)
@@ -21,16 +21,12 @@
       <visual>
         <geometry>
-          <!--<mesh filename="file://$(find robot_table_description)/meshes/robo_table.dae"/>-->
           <mesh filename="package://robot_table_description/meshes/robo_table.dae"/>
         </geometry>
-        <!--<origin xyz="0 0 -0.01" rpy="${pi/2} 0 0"/>-->
         <origin xyz="0 0 0" rpy="${pi/2} 0 0"/>
       </visual>
       <collision>
         <geometry>
-          <!--<mesh filename="file://$(find robot_table_description)/meshes/robo_table.dae"/>-->
           <mesh filename="package://robot_table_description/meshes/robo_table.dae"/>
         </geometry>
-        <!--<origin xyz="0 0 -0.01" rpy="${pi/2} 0 0"/>-->
         <origin xyz="0 0 0" rpy="${pi/2} 0 0"/>
       </collision>
@@ -42,5 +38,4 @@
       <origin xyz="0 0 0.02" rpy="0 0 0" />
     </joint>
-    <!--This will create the specific robot-->
     <xacro:ur_robot
       name="${ur_type}"
@@ -55,5 +50,5 @@
     </xacro:ur_robot>
   </xacro:macro>
-  <!-- Adapter -->
+  <!-- Robot Tool -->
   <xacro:ur_to_robotiq
     prefix=""
